Commit message: URDF that we were using before software update (manually changed Trunk and arms)

File: robot.urdf (robot description, URDF)
Before this commit: robot V23RobotAsm, 30 links, 29 joints
Links:
- added link left_Link1, mass 0.00647716099397792; collision mesh filename=package://V23RobotAsm.SLDASM/meshes/left_Link1.STL; visual mesh filename=package://V23RobotAsm.SLDASM/meshes/left_Link1.STL
- added link left_Link11, mass 0.0127543420299361; collision mesh filename=package://V23RobotAsm.SLDASM/meshes/left_Link11.STL; visual mesh filename=package://V23RobotAsm.SLDASM/meshes/left_Link11.STL
- added link left_Link2, mass 0.00647716099397793; collision mesh filename=package://V23RobotAsm.SLDASM/meshes/left_Link2.STL; visual mesh filename=package://V23RobotAsm.SLDASM/meshes/left_Link2.STL
- added link left_Link22, mass 0.0127543420299362; collision mesh filename=package://V23RobotAsm.SLDASM/meshes/left_Link22.STL; visual mesh filename=package://V23RobotAsm.SLDASM/meshes/left_Link22.STL
- added link left_base_link, mass 0.105853592307918; collision mesh filename=package://V23RobotAsm.SLDASM/meshes/left_base_link.STL; visual mesh filename=package://V23RobotAsm.SLDASM/meshes/left_base_link.STL
- added link right_Link1, mass 0.00647716099397792; collision mesh filename=package://V23RobotAsm.SLDASM/meshes/right_Link1.STL; visual mesh filename=package://V23RobotAsm.SLDASM/meshes/right_Link1.STL
- added link right_Link11, mass 0.0127543420299361; collision mesh filename=package://V23RobotAsm.SLDASM/meshes/right_Link11.STL; visual mesh filename=package://V23RobotAsm.SLDASM/meshes/right_Link11.STL
- added link right_Link2, mass 0.00647716099397793; collision mesh filename=package://V23RobotAsm.SLDASM/meshes/right_Link2.STL; visual mesh filename=package://V23RobotAsm.SLDASM/meshes/right_Link2.STL
- added link right_Link22, mass 0.0127543420299362; collision mesh filename=package://V23RobotAsm.SLDASM/meshes/right_Link22.STL; visual mesh filename=package://V23RobotAsm.SLDASM/meshes/right_Link22.STL
- added link right_base_link, mass 0.105853592307918; collision mesh filename=package://V23RobotAsm.SLDASM/meshes/right_base_link.STL; visual mesh filename=package://V23RobotAsm.SLDASM/meshes/right_base_link.STL
- link left_hand_link: geometry 
- link right_hand_link: geometry 
Joints:
- added joint left_Link1: type fixed, parent left_base_link, child left_Link1, origin xyz=0.036 -0.04 -0.019 rpy=0 0 -0.30719, axis 0 0 1, limit lower=0 upper=1 effort=1 velocity=1
- added joint left_Link11: type fixed, parent left_Link1, child left_Link11, origin xyz=0.042 0 0.003 rpy=0 0 0.30719, axis 0 0 1, limit lower=-1 upper=0 effort=1 velocity=1
- added joint left_Link2: type fixed, parent left_base_link, child left_Link2, origin xyz=0.036 0.04 -0.019 rpy=0 0 0.30719, axis 0 0 1, limit lower=-1 upper=0 effort=1 velocity=1
- added joint left_Link22: type fixed, parent left_Link2, child left_Link22, origin xyz=0.042 0 0.015 rpy=0 0 2.8344, axis 0 0 1, limit lower=0 upper=1 effort=1 velocity=1
- added joint left_base_link: type fixed, parent left_hand_link, child left_base_link, origin xyz=0 0.08 0 rpy=0 0 1.5708
- added joint right_Link1: type fixed, parent right_base_link, child right_Link1, origin xyz=0.036 -0.04 -0.019 rpy=0 0 -0.30719, axis 0 0 1, limit lower=0 upper=1 effort=1 velocity=1
- added joint right_Link11: type fixed, parent right_Link1, child right_Link11, origin xyz=0.042 0 0.003 rpy=0 0 0.30719, axis 0 0 1, limit lower=-1 upper=0 effort=1 velocity=1
- added joint right_Link2: type fixed, parent right_base_link, child right_Link2, origin xyz=0.036 0.04 -0.019 rpy=0 0 0.30719, axis 0 0 1, limit lower=-1 upper=0 effort=1 velocity=1
- added joint right_Link22: type fixed, parent right_Link2, child right_Link22, origin xyz=0.042 0 0.015 rpy=0 0 2.8344, axis 0 0 1, limit lower=0 upper=1 effort=1 velocity=1
- added joint right_base_link: type fixed, parent right_hand_link, child right_base_link, origin xyz=0 -0.084 0 rpy=0 0 -1.5708
- joint AAHead_yaw: origin xyz=0.0625 0 0.243 rpy=0 0 0 -> xyz=0 0 0.243 rpy=0 0 0
- joint Left_Hand_Roll: origin xyz=0.00475 0.07 0.0015 rpy=0 0 0 -> xyz=0 0.07 0.0015 rpy=0 0 0
- joint Left_Shoulder_Pitch: origin xyz=0.0575 0.1063 0.219 rpy=0 0.00088113 0 -> xyz=-0.005 0.1063 0.219 rpy=0 0.00088113 0
- joint Right_Hand_Roll: origin xyz=0.00475 -0.07 0.0015 rpy=0 0 0 -> xyz=0 -0.07 0.0015 rpy=0 0 0
- joint Right_Shoulder_Pitch: origin xyz=0.0575 -0.1063 0.219 rpy=0 0.00088113 0 -> xyz=-0.005 -0.1063 0.219 rpy=0 0.00088113 0
- joint Waist: origin xyz=0.0625 0 -0.1155 rpy=0 0 0 -> xyz=0 0 -0.1155 rpy=0 0 0

Commit message: URDF obtained after updating firmware to version 1.5.1.11

File: robot.urdf (robot description, URDF)
Before this commit: robot V23RobotAsm, 40 links, 39 joints
Links:
- removed link left_Link1
- removed link left_Link11
- removed link left_Link2
- removed link left_Link22
- removed link left_base_link
- removed link right_Link1
- removed link right_Link11
- removed link right_Link2
- removed link right_Link22
- removed link right_base_link
- link AL4: mass 0.2984 -> 0.5570
- link AL5: mass 0.42219 -> 0.43402
- link AL6: mass 0.26532 -> 0.47922
- link AR4: mass 0.3599 -> 0.5570
- link AR6: mass 0.28215 -> 0.47922
- link H2: geometry collision sphere radius=0.08; visual mesh filename=package://V23RobotAsm/meshes/H2.STL
- link Hip_Roll_Left: geometry collision cylinder length=0.16 radius=0.05; visual mesh filename=package://V23RobotAsm/meshes/Hip_Roll_Left.STL
- link Hip_Roll_Right: geometry collision cylinder length=0.16 radius=0.05; visual mesh filename=package://V23RobotAsm/meshes/Hip_Roll_Right.STL
- link Hip_Yaw_Left: geometry collision cylinder length=0.08 radius=0.05; visual mesh filename=package://V23RobotAsm/meshes/Hip_Yaw_Left.STL
- link Hip_Yaw_Right: geometry collision cylinder length=0.08 radius=0.05; visual mesh filename=package://V23RobotAsm/meshes/Hip_Yaw_Right.STL
- link Shank_Left: geometry collision box size=0.1 0.08 0.1; visual mesh filename=package://V23RobotAsm/meshes/Shank_Left.STL
- link Shank_Right: geometry collision box size=0.1 0.08 0.1; visual mesh filename=package://V23RobotAsm/meshes/Shank_Right.STL
- link Trunk: geometry collision box size=0.15 0.2 0.3; visual mesh filename=package://V23RobotAsm/meshes/Trunk.STL
- link left_foot_link: geometry collision box size=0.223 0.1 0.03; visual mesh filename=package://V23RobotAsm/meshes/left_foot_link.STL
- link left_hand_link: mass 0.24875 -> 0.30603; geometry collision mesh filename=package://V23RobotAsm.SLDASM/meshes/AL7.STL; visual mesh filename=package://V23RobotAsm.SLDASM/meshes/AL7.STL
- link right_foot_link: geometry collision box size=0.223 0.1 0.03; visual mesh filename=package://V23RobotAsm/meshes/right_foot_link.STL
- link right_hand_link: mass 0.24612 -> 0.30603; geometry collision mesh filename=package://V23RobotAsm.SLDASM/meshes/AR7.STL; visual mesh filename=package://V23RobotAsm.SLDASM/meshes/AR7.STL
Joints:
- removed joint Waist
- removed joint left_Link1
- removed joint left_Link11
- removed joint left_Link2
- removed joint left_Link22
- removed joint left_base_link
- removed joint right_Link1
- removed joint right_Link11
- removed joint right_Link2
- removed joint right_Link22
- removed joint right_base_link
- added joint Waist_Joint: type revolute, parent Trunk, child Waist, origin xyz=0.0625 0 -0.1155 rpy=0 0 0, axis 0 0 1, limit lower=-1.57 upper=1.57 effort=30 velocity=10.88
- joint AAHead_yaw: limit lower=0 upper=0 effort=0 velocity=0 -> lower=-1.57 upper=1.57 effort=7 velocity=12.56; origin xyz=0 0 0.243 rpy=0 0 0 -> xyz=0.0625 0 0.243 rpy=0 0 0
- joint Head_pitch: limit lower=0 upper=0 effort=0 velocity=0 -> lower=-0.35 upper=1.22 effort=7 velocity=12.56
- joint Left_Ankle_Pitch: limit lower=0 upper=0 effort=0 velocity=0 -> lower=-0.87 upper=0.35 effort=12 velocity=18.8
- joint Left_Ankle_Roll: limit lower=0 upper=0 effort=0 velocity=0 -> lower=-0.44 upper=0.44 effort=12 velocity=12.4
- joint Left_Elbow_Pitch: limit lower=0 upper=0 effort=0 velocity=0 -> lower=-2.234 upper=2.234 effort=18 velocity=18.84
- joint Left_Elbow_Yaw: limit lower=0 upper=0 effort=0 velocity=0 -> lower=-2.1402 upper=1.6844 effort=18 velocity=18.84
- joint Left_Hand_Roll: limit lower=0 upper=0 effort=0 velocity=0 -> lower=-1.3614 upper=1.4285 effort=7 velocity=12.56; origin xyz=0 0.07 0.0015 rpy=0 0 0 -> xyz=0.00475 0.07 0.0015 rpy=0 0 0
- joint Left_Hip_Pitch: limit lower=0 upper=0 effort=0 velocity=0 -> lower=-1.8 upper=1.57 effort=45 velocity=12.5
- joint Left_Hip_Roll: limit lower=0 upper=0 effort=0 velocity=0 -> lower=-0.3 upper=1.57 effort=30 velocity=10.9
- joint Left_Hip_Yaw: limit lower=0 upper=0 effort=0 velocity=0 -> lower=-1 upper=1 effort=30 velocity=10.9
- joint Left_Knee_Pitch: limit lower=0 upper=0 effort=0 velocity=0 -> lower=0 upper=2.34 effort=60 velocity=11.7
- joint Left_Shoulder_Pitch: limit lower=0 upper=0 effort=0 velocity=0 -> lower=-3.29 upper=1.18 effort=18 velocity=18.84; origin xyz=-0.005 0.1063 0.219 rpy=0 0.00088113 0 -> xyz=0.0575 0.1063 0.219 rpy=0 0.00088113 0
- joint Left_Shoulder_Roll: limit lower=0 upper=0 effort=0 velocity=0 -> lower=-1.577 upper=1.7055 effort=18 velocity=18.84
- joint Left_Wrist_Pitch: limit lower=0 upper=0 effort=0 velocity=0 -> lower=-2.5821 upper=2.5821 effort=7 velocity=12.56
- joint Left_Wrist_Yaw: limit lower=0 upper=0 effort=0 velocity=0 -> lower=-1.8185 upper=1.4261 effort=18 velocity=18.84
- joint Right_Ankle_Pitch: limit lower=0 upper=0 effort=0 velocity=0 -> lower=-0.87 upper=0.35 effort=12 velocity=18.8
- joint Right_Ankle_Roll: limit lower=0 upper=0 effort=0 velocity=0 -> lower=-0.44 upper=0.44 effort=12 velocity=12.4
- joint Right_Elbow_Pitch: limit lower=0 upper=0 effort=0 velocity=0 -> lower=-2.234 upper=2.234 effort=18 velocity=18.84
- joint Right_Elbow_Yaw: limit lower=0 upper=0 effort=0 velocity=0 -> lower=-1.6844 upper=2.1402 effort=18 velocity=18.84
- joint Right_Hand_Roll: limit lower=0 upper=0 effort=0 velocity=0 -> lower=-1.4285 upper=1.3614 effort=7 velocity=12.56; origin xyz=0 -0.07 0.0015 rpy=0 0 0 -> xyz=0.00475 -0.07 0.0015 rpy=0 0 0
- joint Right_Hip_Pitch: limit lower=0 upper=0 effort=0 velocity=0 -> lower=-1.8 upper=1.57 effort=45 velocity=12.5
- joint Right_Hip_Roll: limit lower=0 upper=0 effort=0 velocity=0 -> lower=-1.57 upper=0.3 effort=30 velocity=10.9
- joint Right_Hip_Yaw: limit lower=0 upper=0 effort=0 velocity=0 -> lower=-1 upper=1 effort=30 velocity=10.9
- joint Right_Knee_Pitch: limit lower=0 upper=0 effort=0 velocity=0 -> lower=0 upper=2.34 effort=60 velocity=11.7
- joint Right_Shoulder_Pitch: limit lower=0 upper=0 effort=0 velocity=0 -> lower=-3.29 upper=1.1868 effort=18 velocity=18.84; origin xyz=-0.005 -0.1063 0.219 rpy=0 0.00088113 0 -> xyz=0.0575 -0.1063 0.219 rpy=0 0.00088113 0
- joint Right_Shoulder_Roll: limit lower=0 upper=0 effort=0 velocity=0 -> lower=-1.7055 upper=1.577 effort=18 velocity=18.84
- joint Right_Wrist_Pitch: limit lower=0 upper=0 effort=0 velocity=0 -> lower=-2.5821 upper=2.5821 effort=7 velocity=12.56
- joint Right_Wrist_Yaw: limit lower=0 upper=0 effort=0 velocity=0 -> lower=-1.4261 upper=1.8185 effort=18 velocity=18.84

Commit message: Change Waist_Joint to Waist to match joint_states

File: robot.urdf (robot description, URDF)
Before this commit: robot V23RobotAsm, 30 links, 29 joints
Joints:
- removed joint Waist_Joint
- added joint Waist: type revolute, parent Trunk, child Waist, origin xyz=0.0625 0 -0.1155 rpy=0 0 0, axis 0 0 1, limit lower=-1.57 upper=1.57 effort=30 velocity=10.88

Commit message: Changes to urdf to add left_Link* and right_Link*

File: robot.urdf (robot description, URDF)
Before this commit: robot V23RobotAsm, 30 links, 29 joints
Links:
- added link left_Link1, mass 0.00647716099397792; collision mesh filename=package://V23RobotAsm.SLDASM/meshes/left_Link1.STL; visual mesh filename=package://V23RobotAsm.SLDASM/meshes/left_Link1.STL
- added link left_Link11, mass 0.0127543420299361; collision mesh filename=package://V23RobotAsm.SLDASM/meshes/left_Link11.STL; visual mesh filename=package://V23RobotAsm.SLDASM/meshes/left_Link11.STL
- added link left_Link2, mass 0.00647716099397793; collision mesh filename=package://V23RobotAsm.SLDASM/meshes/left_Link2.STL; visual mesh filename=package://V23RobotAsm.SLDASM/meshes/left_Link2.STL
- added link left_Link22, mass 0.0127543420299362; collision mesh filename=package://V23RobotAsm.SLDASM/meshes/left_Link22.STL; visual mesh filename=package://V23RobotAsm.SLDASM/meshes/left_Link22.STL
- added link left_base_link, mass 0.105853592307918; collision mesh filename=package://V23RobotAsm.SLDASM/meshes/left_base_link.STL; visual mesh filename=package://V23RobotAsm.SLDASM/meshes/left_base_link.STL
- added link right_Link1, mass 0.00647716099397792; collision mesh filename=package://V23RobotAsm.SLDASM/meshes/right_Link1.STL; visual mesh filename=package://V23RobotAsm.SLDASM/meshes/right_Link1.STL
- added link right_Link11, mass 0.0127543420299361; collision mesh filename=package://V23RobotAsm.SLDASM/meshes/right_Link11.STL; visual mesh filename=package://V23RobotAsm.SLDASM/meshes/right_Link11.STL
- added link right_Link2, mass 0.00647716099397793; collision mesh filename=package://V23RobotAsm.SLDASM/meshes/right_Link2.STL; visual mesh filename=package://V23RobotAsm.SLDASM/meshes/right_Link2.STL
- added link right_Link22, mass 0.0127543420299362; collision mesh filename=package://V23RobotAsm.SLDASM/meshes/right_Link22.STL; visual mesh filename=package://V23RobotAsm.SLDASM/meshes/right_Link22.STL
- added link right_base_link, mass 0.105853592307918; collision mesh filename=package://V23RobotAsm.SLDASM/meshes/right_base_link.STL; visual mesh filename=package://V23RobotAsm.SLDASM/meshes/right_base_link.STL
- link left_hand_link: mass 0.30603 -> 0.24875; geometry 
- link right_hand_link: mass 0.30603 -> 0.24612; geometry 
Joints:
- added joint left_Link1: type fixed, parent left_base_link, child left_Link1, origin xyz=0.036 -0.04 -0.019 rpy=0 0 -0.30719, axis 0 0 1, limit lower=0 upper=1 effort=1 velocity=1
- added joint left_Link11: type fixed, parent left_Link1, child left_Link11, origin xyz=0.042 0 0.003 rpy=0 0 0.30719, axis 0 0 1, limit lower=-1 upper=0 effort=1 velocity=1
- added joint left_Link2: type fixed, parent left_base_link, child left_Link2, origin xyz=0.036 0.04 -0.019 rpy=0 0 0.30719, axis 0 0 1, limit lower=-1 upper=0 effort=1 velocity=1
- added joint left_Link22: type fixed, parent left_Link2, child left_Link22, origin xyz=0.042 0 0.015 rpy=0 0 2.8344, axis 0 0 1, limit lower=0 upper=1 effort=1 velocity=1
- added joint left_base_link: type fixed, parent left_hand_link, child left_base_link, origin xyz=0 0.08 0 rpy=0 0 1.5708
- added joint right_Link1: type fixed, parent right_base_link, child right_Link1, origin xyz=0.036 -0.04 -0.019 rpy=0 0 -0.30719, axis 0 0 1, limit lower=0 upper=1 effort=1 velocity=1
- added joint right_Link11: type fixed, parent right_Link1, child right_Link11, origin xyz=0.042 0 0.003 rpy=0 0 0.30719, axis 0 0 1, limit lower=-1 upper=0 effort=1 velocity=1
- added joint right_Link2: type fixed, parent right_base_link, child right_Link2, origin xyz=0.036 0.04 -0.019 rpy=0 0 0.30719, axis 0 0 1, limit lower=-1 upper=0 effort=1 velocity=1
- added joint right_Link22: type fixed, parent right_Link2, child right_Link22, origin xyz=0.042 0 0.015 rpy=0 0 2.8344, axis 0 0 1, limit lower=0 upper=1 effort=1 velocity=1
- added joint right_base_link: type fixed, parent right_hand_link, child right_base_link, origin xyz=0 -0.084 0 rpy=0 0 -1.5708

Commit message: this is the robot urdf right before updating the firmware again. Probably wrong

File: robot.urdf (robot description, URDF)
Before this commit: robot V23RobotAsm, 40 links, 39 joints
Joints:
- joint Left_Wrist_Pitch: origin xyz=0 0.105 0.00025 rpy=0 0 0 -> xyz=0 0.105 0.00025 rpy=0 0.19 0
- joint Right_Wrist_Pitch: origin xyz=0 -0.105 0.00025 rpy=0 0 0 -> xyz=0 -0.105 0.00025 rpy=0 0.19 0

Commit message: urdf obtained after updating the firmware

File: robot.urdf (robot description, URDF)
Before this commit: robot V23RobotAsm, 40 links, 39 joints
Links:
- removed link left_Link1
- removed link left_Link11
- removed link left_Link2
- removed link left_Link22
- removed link left_base_link
- removed link right_Link1
- removed link right_Link11
- removed link right_Link2
- removed link right_Link22
- removed link right_base_link
- link left_hand_link: mass 0.24875 -> 0.30603; geometry collision mesh filename=package://V23RobotAsm.SLDASM/meshes/AL7.STL; visual mesh filename=package://V23RobotAsm.SLDASM/meshes/AL7.STL
- link right_hand_link: mass 0.24612 -> 0.30603; geometry collision mesh filename=package://V23RobotAsm.SLDASM/meshes/AR7.STL; visual mesh filename=package://V23RobotAsm.SLDASM/meshes/AR7.STL
Joints:
- removed joint Waist
- removed joint left_Link1
- removed joint left_Link11
- removed joint left_Link2
- removed joint left_Link22
- removed joint left_base_link
- removed joint right_Link1
- removed joint right_Link11
- removed joint right_Link2
- removed joint right_Link22
- removed joint right_base_link
- added joint Waist_Joint: type revolute, parent Trunk, child Waist, origin xyz=0.0625 0 -0.1155 rpy=0 0 0, axis 0 0 1, limit lower=-1.57 upper=1.57 effort=30 velocity=10.88
- joint Left_Wrist_Pitch: origin xyz=0 0.105 0.00025 rpy=0 0.19 0 -> xyz=0 0.105 0.00025 rpy=0 0 0
- joint Right_Wrist_Pitch: origin xyz=0 -0.105 0.00025 rpy=0 0.19 0 -> xyz=0 -0.105 0.00025 rpy=0 0 0

Commit message: urdf on v1.6.1

File: robot.urdf (robot description, URDF)
Before this commit: robot V23RobotAsm, 30 links, 29 joints
Links:
- link AL1: geometry collision mesh filename=file:///opt/booster/Gait/configs/T1_7DofArm/T1_release_mesh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; visual mesh filename=file:///opt/booster/Gait/configs/T1_7DofArm/T1_release_mesh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
- link AL2: geometry collision mesh filename=file:///opt/booster/Gait/configs/T1_7DofArm/T1_release_mesh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; visual mesh filename=file:///opt/booster/Gait/configs/T1_7DofArm/T1_release_mesh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
- link AL3: geometry collision mesh filename=file:///opt/booster/Gait/configs/T1_7DofArm/T1_release_mesh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; visual mesh filename=file:///opt/booster/Gait/configs/T1_7DofArm/T1_release_mesh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
- link AR1: geometry collision mesh filename=file:///opt/booster/Gait/configs/T1_7DofArm/T1_release_mesh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; visual mesh filename=file:///opt/booster/Gait/configs/T1_7DofArm/T1_release_mesh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
- link AR2: geometry collision mesh filename=file:///opt/booster/Gait/configs/T1_7DofArm/T1_release_mesh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; visual mesh filename=file:///opt/booster/Gait/configs/T1_7DofArm/T1_release_mesh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
- link AR3: geometry collision mesh filename=file:///opt/booster/Gait/configs/T1_7DofArm/T1_release_mesh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; visual mesh filename=file:///opt/booster/Gait/configs/T1_7DofArm/T1_release_mesh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
- link Ankle_Cross_Left: geometry collision mesh filename=file:///opt/booster/Gait/configs/T1_7DofArm/T1_release_mesh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; visual mesh filename=file:///opt/booster/Gait/configs/T1_7DofArm/T1_release_mesh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
- link Ankle_Cross_Right: geometry collision mesh filename=file:///opt/booster/Gait/configs/T1_7DofArm/T1_release_mesh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; visual mesh filename=file:///opt/booster/Gait/configs/T1_7DofArm/T1_release_mesh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
- link H1: geometry collision mesh filename=file:///opt/booster/Gait/configs/T1_7DofArm/T1_release_mesh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; visual mesh filename=file:///opt/booster/Gait/configs/T1_7DofArm/T1_release_mesh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
- link H2: geometry collision sphere radius=0.08; visual mesh filename=file:///opt/booster/Gait/configs/T1_7DofArm/T1_release_mesh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
- link Hip_Pitch_Left: geometry collision mesh filename=file:///opt/booster/Gait/configs/T1_7DofArm/T1_release_mesh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; visual mesh filename=file:///opt/booster/Gait/configs/T1_7DofArm/T1_release_mesh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
- link Hip_Pitch_Right: geometry collision mesh filename=file:///opt/booster/Gait/configs/T1_7DofArm/T1_release_mesh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; visual mesh filename=file:///opt/booster/Gait/configs/T1_7DofArm/T1_release_mesh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
- link Hip_Roll_Left: geometry collision cylinder length=0.16 radius=0.05; visual mesh filename=file:///opt/booster/Gait/configs/T1_7DofArm/T1_release_mesh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
- link Hip_Roll_Right: geometry collision cylinder length=0.16 radius=0.05; visual mesh filename=file:///opt/booster/Gait/configs/T1_7DofArm/T1_release_mesh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
- link Hip_Yaw_Left: geometry collision cylinder length=0.08 radius=0.05; visual mesh filename=file:///opt/booster/Gait/configs/T1_7DofArm/T1_release_mesh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
- link Hip_Yaw_Right: geometry collision cylinder length=0.08 radius=0.05; visual mesh filename=file:///opt/booster/Gait/configs/T1_7DofArm/T1_release_mesh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
- link Shank_Left: geometry collision box size=0.1 0.08 0.1; visual mesh filename=file:///opt/booster/Gait/configs/T1_7DofArm/T1_release_mesh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
- link Shank_Right: geometry collision box size=0.1 0.08 0.1; visual mesh filename=file:///opt/booster/Gait/configs/T1_7DofArm/T1_release_mesh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
- link Trunk: geometry collision box size=0.15 0.2 0.3; visual mesh filename=file:///opt/booster/Gait/configs/T1_7DofArm/T1_release_mesh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
- link Waist: geometry collision mesh filename=file:///opt/booster/Gait/configs/T1_7DofArm/T1_release_mesh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; visual mesh filename=file:///opt/booster/Gait/configs/T1_7DofArm/T1_release_mesh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
- link left_foot_link: geometry collision box size=0.223 0.1 0.03; visual mesh filename=file:///opt/booster/Gait/configs/T1_7DofArm/T1_release_mesh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
- link right_foot_link: geometry collision box size=0.223 0.1 0.03; visual mesh filename=file:///opt/booster/Gait/configs/T1_7DofArm/T1_release_mesh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
Joints:
- removed joint Waist
- added joint Waist_Joint: type revolute, parent Trunk, child Waist, origin xyz=0.0625 0 -0.1155 rpy=0 0 0, axis 0 0 1, limit lower=-1.57 upper=1.57 effort=30 velocity=10.88
- joint Left_Wrist_Pitch: origin xyz=0 0.105 0.00025 rpy=0 0.19 0 -> xyz=0 0.105 0.00025 rpy=0 0 0
- joint Right_Wrist_Pitch: origin xyz=0 -0.105 0.00025 rpy=0 0.19 0 -> xyz=0 -0.105 0.00025 rpy=0 0 0
